File: RPiOperant.sch (EAGLE design)
At the start: 44 parts, among them IC1 74LS14N, IC2 MCP3202P, J1 RASPBERRYPI-40-PIN-GPIO_PTH_N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, J2 POWER_JACK, J3 POWER_JACK

Commit message: update traces
Connections:
- net 3.3V renamed +3V3
- net 5V renamed +5V

Commit message: rework
Parts:
- removed IC2: MCP3202P, microchip:MCP3202P
- removed J1: RASPBERRYPI-40-PIN-GPIO_PTH_NO_SHROUD, SparkFun-Connectors:RASPBERRYPI-40-PIN-GPIO_PTH_NO_SHROUD
- removed J10, J11, J12, J13, J14, J15, J16, J17, J18, J4, J5, J6, J7, J8, J9: (no value), SparkFun-Connectors:CONN_022.54MM_SCREWTERM
- removed R13, R14, R15: 330, resistor:R-US_0207/7
- added IC3: MCP3008, adafruit:MCP3008
- added SV1, SV2: (no value), con-lstb:MA20-2
- added X1: (no value), con-subd:F25HP
Connections:
- removed net N$1: IC1A.O, J1.GP5
- removed net N$11: J7.2, R7.1, R8.1
- removed net N$13: J8.1, R9.1
- removed net N$14: J9.1, R10.1
- removed net N$15: J10.1, R11.1
- removed net N$16: J11.1, R12.1
- removed net N$17: J12.1, R13.2
- removed net N$18: J13.1, R14.2
- removed net N$19: J14.1, R15.2
- removed net N$2: IC1B.O, J1.GP6
- removed net N$20: J1.GP22, R13.1
- removed net N$21: J1.GP27, R14.1
- removed net N$22: J1.GP17, R15.1
- removed net N$23: D1.A, J15.2, Q1.D
- removed net N$25: J1.GP16, R16.1
- removed net N$26: D2.A, J16.2, Q2.D
- removed net N$28: J1.GP12, R17.1
- removed net N$29: IC2.!CS!/SHDN, J1.CE0
- removed net N$3: IC1C.O, J1.GP13
- removed net N$30: IC2.CLK, J1.SCLK
- removed net N$31: IC2.DOUT, J1.MISO
- removed net N$32: IC2.DIN, J1.MOSI
- removed net N$33: IC2.CH0, U1.VOUT
- removed net N$34: J1.GP25, J17.2
- removed net N$35: J1.GP24, J17.1
- removed net N$36: J1.SCL, J18.2
- removed net N$37: J1.SDA, J18.1
- removed net N$4: IC1D.O, J1.GP26
- removed net N$5: J4.2, R1.1, R2.1
- removed net N$7: J5.2, R3.1, R4.1
- removed net N$9: J6.2, R5.1, R6.1
- new net CE0: SV1.24
- new net CE1: IC3./CS, SV1.26
- new net CENTER_IR: X1.11
- new net CENTER_LED: X1.8
- new net CENTER_PECK_GPIO: IC1C.O, SV1.33
- new net CENTNER_IR: R5.1, R6.1
- new net GPIO2: SV1.3, X1.14
- new net GPIO20: X1.21
- new net GPIO21: X1.22
- new net GPIO23: X1.16
- new net GPIO24: X1.17
- new net GPIO25: X1.18
- new net GPIO3: SV1.5, X1.15
- new net GPIO4: SV1.7
- new net GPIO7: X1.20
- new net GPIO8: X1.19
- new net HOPPER: D1.A, Q1.D, X1.6
- new net HOPPER_IR: R1.1, R2.1, X1.13
- new net HOPPER_IR_GPIO: IC1A.O, SV1.29
- new net HOPPER_TRIG_GPIO: R16.1, SV1.36
- new net HOUSE_LIGHTS: D2.A, Q2.D, X1.5
- new net LEFT_IR: R3.1, R4.1, X1.12
- new net LEFT_LED: X1.9
- new net LEFT_PECK_GPIO: IC1B.O, SV1.31
- new net LIGHTS_TRIG_GPIO: R17.1, SV1.32
- new net MISO: IC3.DOUT, SV1.21
- new net MOSI: IC3.DIN, SV1.19
- new net N$47: X1.4
- new net N$48: X1.3
- new net N$49: X1.2
- new net N$50: X1.1
- new net RIGHT_IR: R7.1, R8.1, X1.10
- new net RIGHT_LED: X1.7
- new net RIGHT_PECK_GPIO: IC1D.O, SV1.37
- new net SCLK: IC3.CLK, SV1.23
- net +3V3: now also IC3.VDD, IC3.VREF; no longer IC2.VDD/VREF, U1.VCC
- net +5V: now also X1.25
- net 12V: now also X1.24; no longer J15.1, J16.1
- net GND: now also IC3.AGND, IC3.GND, X1.23, X1.G1, X1.G2; no longer IC2.VSS, J1.GND@14, J1.GND@20, J1.GND@25, J1.GND@30, J1.GND@34, J1.GND@39, J1.GND@6, J1.GND@9, J10.2, J11.2, J12.2, J13.2, J14.2, J4.1, J5.1, J6.1, J7.1, J8.2, J9.2, U1.GND
Other:
- note removed: "CENTER LED"
- note removed: "HOPPER IR SENSE"
- note removed: "LEFT LED"
- note removed: "RIGHT LED"
- moved on the sheet: D1, D2, IC1A, IC1B, IC1C, IC1D, IC1P, Q1, Q2, R1, R16, R17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

Commit message: new board
Parts:
- removed R10, R11, R12, R9: 330, resistor:R-US_0207/7
- added R13, R14: 1k, resistor:R-US_0207/7
- added R15, R20: 4.3, resistor:R-US_0207/7
- added R21, R22, R23: 330, resistor:R-US_0207/7
- IC1: SPICEPREFIX (none) -> I
- R3, R4: SPICEPREFIX (none) -> R
Connections:
- removed net GPIO23: X1.16
- removed net GPIO24: X1.17
- removed net N$47: X1.4
- removed net N$48: X1.3
- removed net N$49: X1.2
- removed net N$50: X1.1
- new net ADC0: IC3.CH0, X1.2
- new net ADC1: IC3.CH1, X1.1
- new net ADC2: IC3.CH2, X1.17
- new net ADC3: IC3.CH3
- new net ADC4: IC3.CH4, X1.16
- new net ADC5: IC3.CH5
- new net ADC6: IC3.CH6
- new net ADC7: IC3.CH7
- new net GPIO17: R23.1, SV1.11, SV2.11
- new net GPIO22: R21.1, SV1.15, SV2.15
- new net GPIO27: R22.2, SV1.13, SV2.13
- new net IR_1: R13.1, R15.1, X1.4
- new net IR_1_GPIO: IC1E.O
- new net IR_2: R14.1, R20.1, X1.3
- new net IR_2_GPIO: IC1F.O
- new net N$1: IC1E.I, R13.2
- new net N$2: IC1F.I, R14.2
- net +3V3: now also R15.2, R20.2; no longer R10.2, R11.2, R12.2, R9.2
- net CE0: now also SV2.24
- net CE1: now also SV2.26
- net CENTER_LED: now also R22.1
- net CENTER_PECK_GPIO: now also SV2.33
- net GND: now also SV1.14, SV1.20, SV1.25, SV1.30, SV1.34, SV1.39, SV1.6, SV1.9, SV2.14, SV2.20, SV2.25, SV2.30, SV2.34, SV2.39, SV2.6, SV2.9
- net GPIO2: now also SV2.3
- net GPIO3: now also SV2.5
- net GPIO4: now also SV2.7
- net HOPPER_IR_GPIO: now also SV2.29
- net HOPPER_TRIG_GPIO: now also SV2.36
- net LEFT_LED: now also R23.2
- net LEFT_PECK_GPIO: now also SV2.31
- net LIGHTS_TRIG_GPIO: now also SV2.32
- net MISO: now also SV2.21
- net MOSI: now also SV2.19
- net RIGHT_LED: now also R21.2
- net RIGHT_PECK_GPIO: now also SV2.37
- net SCLK: now also SV2.23
Other:
- moved on the sheet: D1, D2, IC1B, IC1C, IC1D, Q1, Q2, R16, R17, R2, R3, R4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

Commit message: updates
Parts:
- removed U1: (no value), SparkFun-Sensors:TMP36GT9
Connections:
- new net RPI_3.3V: SV1.1, SV1.17, SV2.1, SV2.17
- new net RPI_5V: SV1.2, SV1.4, SV2.2, SV2.4
- net IR_1_GPIO: now also SV1.16
- net IR_2_GPIO: now also SV1.18, SV2.18
Other:
- moved on the sheet: D1, D2, IC3, Q1, Q2, R16, R17

Commit message: panel breakeout :
Parts:
- added R10, R11, R12, R9: 330, resistor:R-US_0207/7
Connections:
- removed net GPIO20: X1.21
- removed net GPIO21: X1.22
- removed net GPIO7: X1.20
- removed net GPIO8: X1.19
- new net HOPPER_IR_LED: R12.1, X1.19
- new net IR_LED_C: R10.1, X1.21
- new net IR_LED_L: R9.1, X1.22
- new net IR_LED_R: R11.1, X1.20
- net +3V3: now also R10.2, R11.2, R12.2, R9.2
Changed lines of the file:
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@@
 <part name="GND5" library="SparkFun-PowerSymbols" deviceset="GND" device=""/>
 <part name="GND6" library="SparkFun-PowerSymbols" deviceset="GND" device=""/>
+<part name="R9" library="resistor" library_urn="urn:adsk.eagle:library:348" deviceset="R-US_" device="0207/7" package3d_urn="urn:adsk.eagle:package:25942/1" value="330"/>
+<part name="R10" library="resistor" library_urn="urn:adsk.eagle:library:348" deviceset="R-US_" device="0207/7" package3d_urn="urn:adsk.eagle:package:25942/1" value="330"/>
+<part name="R11" library="resistor" library_urn="urn:adsk.eagle:library:348" deviceset="R-US_" device="0207/7" package3d_urn="urn:adsk.eagle:package:25942/1" value="330"/>
+<part name="+3V8" library="supply1" library_urn="urn:adsk.eagle:library:371" deviceset="+3V3" device=""/>
+<part name="R12" library="resistor" library_urn="urn:adsk.eagle:library:348" deviceset="R-US_" device="0207/7" package3d_urn="urn:adsk.eagle:package:25942/1" value="330"/>
 </parts>
 <sheets>
@@
 <instance part="GND5" gate="1" x="96.52" y="22.86"/>
 <instance part="GND6" gate="1" x="119.38" y="22.86"/>
+<instance part="R9" gate="G$1" x="134.62" y="144.78" rot="R180"/>
+<instance part="R10" gate="G$1" x="134.62" y="134.62" rot="R180"/>
+<instance part="R11" gate="G$1" x="134.62" y="124.46" rot="R180"/>
+<instance part="+3V8" gate="G$1" x="124.46" y="152.4"/>
+<instance part="R12" gate="G$1" x="134.62" y="114.3" rot="R180"/>
 </instances>
 <busses>
@@
 </segment>
 </net>
-<net name="GPIO21" class="0">
-<segment>
-<pinref part="X1" gate="G$1" pin="22"/>
-<wire x1="-111.76" y1="129.54" x2="-111.76" y2="121.92" width="0.1524" layer="91"/>
-<label x="-111.76" y="121.92" size="1.016" layer="91" rot="R270" xref="yes"/>
-</segment>
-</net>
-<net name="GPIO20" class="0">
-<segment>
-<pinref part="X1" gate="G$1" pin="21"/>
-<wire x1="-109.22" y1="129.54" x2="-109.22" y2="121.92" width="0.1524" layer="91"/>
-<label x="-109.22" y="121.92" size="1.016" layer="91" rot="R270" xref="yes"/>
-</segment>
-</net>
-<net name="GPIO7" class="0">
-<segment>
-<pinref part="X1" gate="G$1" pin="20"/>
-<wire x1="-106.68" y1="129.54" x2="-106.68" y2="121.92" width="0.1524" layer="91"/>
-<label x="-106.68" y="121.92" size="1.016" layer="91" rot="R270" xref="yes"/>
-</segment>
-</net>
-<net name="GPIO8" class="0">
-<segment>
-<pinref part="X1" gate="G$1" pin="19"/>
-<wire x1="-104.14" y1="129.54" x2="-104.14" y2="121.92" width="0.1524" layer="91"/>
-<label x="-104.14" y="121.92" size="1.016" layer="91" rot="R270" xref="yes"/>
-</segment>
-</net>
 <net name="GPIO25" class="0">
 <segment>
@@
 <pinref part="R20" gate="G$1" pin="2"/>
 <wire x1="-167.64" y1="-35.56" x2="-167.64" y2="-38.1" width="0.1524" layer="91"/>
+</segment>
+<segment>
+<pinref part="R11" gate="G$1" pin="2"/>
+<wire x1="129.54" y1="124.46" x2="124.46" y2="124.46" width="0.1524" layer="91"/>
+<wire x1="124.46" y1="124.46" x2="124.46" y2="134.62" width="0.1524" layer="91"/>
+<pinref part="R9" gate="G$1" pin="2"/>
+<wire x1="124.46" y1="134.62" x2="124.46" y2="144.78" width="0.1524" layer="91"/>
+<wire x1="124.46" y1="144.78" x2="124.46" y2="149.86" width="0.1524" layer="91"/>
+<wire x1="129.54" y1="144.78" x2="124.46" y2="144.78" width="0.1524" layer="91"/>
+<junction x="124.46" y="144.78"/>
+<pinref part="R10" gate="G$1" pin="2"/>
+<wire x1="129.54" y1="134.62" x2="124.46" y2="134.62" width="0.1524" layer="91"/>
+<junction x="124.46" y="134.62"/>
+<pinref part="+3V8" gate="G$1" pin="+3V3"/>
+<pinref part="R12" gate="G$1" pin="2"/>
+<wire x1="129.54" y1="114.3" x2="124.46" y2="114.3" width="0.1524" layer="91"/>
+<wire x1="124.46" y1="114.3" x2="124.46" y2="124.46" width="0.1524" layer="91"/>
+<junction x="124.46" y="124.46"/>
 </segment>
 </net>
@@
 </segment>
 </net>
+<net name="IR_LED_L" class="0">
+<segment>
+<pinref part="X1" gate="G$1" pin="22"/>
+<wire x1="-111.76" y1="129.54" x2="-111.76" y2="121.92" width="0.1524" layer="91"/>
+<label x="-111.76" y="121.92" size="1.016" layer="91" rot="R270" xref="yes"/>
+</segment>
+<segment>
+<pinref part="R9" gate="G$1" pin="1"/>
+<wire x1="139.7" y1="144.78" x2="147.32" y2="144.78" width="0.1524" layer="91"/>
+<label x="147.32" y="144.78" size="1.016" layer="91" xref="yes"/>
+</segment>
+</net>
+<net name="IR_LED_C" class="0">
+<segment>
+<pinref part="X1" gate="G$1" pin="21"/>
+<wire x1="-109.22" y1="129.54" x2="-109.22" y2="121.92" width="0.1524" layer="91"/>
+<label x="-109.22" y="121.92" size="1.016" layer="91" rot="R270" xref="yes"/>
+</segment>
+<segment>
+<pinref part="R10" gate="G$1" pin="1"/>
+<wire x1="139.7" y1="134.62" x2="147.32" y2="134.62" width="0.1524" layer="91"/>
+<label x="147.32" y="134.62" size="1.016" layer="91" xref="yes"/>
+</segment>
+</net>
+<net name="IR_LED_R" class="0">
+<segment>
+<pinref part="X1" gate="G$1" pin="20"/>
+<wire x1="-106.68" y1="129.54" x2="-106.68" y2="121.92" width="0.1524" layer="91"/>
+<label x="-106.68" y="121.92" size="1.016" layer="91" rot="R270" xref="yes"/>
+</segment>
+<segment>
+<pinref part="R11" gate="G$1" pin="1"/>
+<wire x1="139.7" y1="124.46" x2="147.32" y2="124.46" width="0.1524" layer="91"/>
+<label x="147.32" y="124.46" size="1.016" layer="91" xref="yes"/>
+</segment>
+</net>
+<net name="HOPPER_IR_LED" class="0">
+<segment>
+<pinref part="X1" gate="G$1" pin="19"/>
+<wire x1="-104.14" y1="129.54" x2="-104.14" y2="121.92" width="0.1524" layer="91"/>
+<label x="-104.14" y="121.92" size="1.016" layer="91" rot="R270" xref="yes"/>
+</segment>
+<segment>
+<pinref part="R12" gate="G$1" pin="1"/>
+<wire x1="139.7" y1="114.3" x2="147.32" y2="114.3" width="0.1524" layer="91"/>
+<label x="147.32" y="114.3" size="1.016" layer="91" xref="yes"/>
+</segment>
+</net>

Commit message: new schematic
Parts:
- removed D2: 1N4004, diode:1N4004
- removed Q2: (no value), adafruit:MOSFET-NGDS_TO220V
- removed R22, R23: 330, resistor:R-US_0207/7
- added IC2: 74LS14N, 74xx-us:74LS14N
- added J1, J4: USB_B_PTH, SparkFun-Connectors:USB_B_PTH
- added J5, J6, J7, J8, J9: 1X2-3.5MM, adafruit:1X2-3.5MM
- added Q3, Q4, Q5, Q6: (no value), adafruit:MOSFET-NGDS_TO220V
- added R24, R25, R26, R27, R28, R29: 1k, resistor:R-US_0207/7
- added R30, R31, R32, R33, R34, R35: 4.3k, resistor:R-US_0207/7
- added R36, R37, R38: 330, resistor:R-US_0207/7
- added U1: (no value), adafruit:PCA9685
- added X2: (no value), con-subd:F25HP
- R17: value 1k -> 330
Connections:
- removed net GPIO2: SV1.3, SV2.3, X1.14
- removed net GPIO25: X1.18
- removed net GPIO3: SV1.5, SV2.5, X1.15
- removed net GPIO4: SV1.7, SV2.7
- removed net HOPPER_IR_LED: R12.1, X1.19
- removed net HOUSE_LIGHTS: D2.A, Q2.D, X1.5
- removed net IR_LED_C: R10.1, X1.21
- removed net IR_LED_L: R9.1, X1.22
- removed net IR_LED_R: R11.1, X1.20
- removed net LIGHTS_TRIG_GPIO: R17.1, SV1.32, SV2.32
- new net AUX1: J5.1, SV1.7, X2.1
- new net AUX2: J5.2, SV1.32, X2.2
- new net AUX3: J6.1, X2.3
- new net AUX4: J6.2, X2.4
- new net CENTNER_LED: R36.1
- new net GPIO18: J9.2, SV1.12
- new net HOUSELIGHT_B: Q4.D, X1.20
- new net HOUSELIGHT_B_GPIO: Q4.G, U1.PWM2
- new net HOUSELIGHT_G: Q5.D, X1.21
- new net HOUSELIGHT_G_GPIO: Q5.G, U1.PWM1
- new net HOUSELIGHT_R: Q3.D, X1.22
- new net HOUSELIGHT_R_GPIO: Q3.G, U1.PWM0
- new net HOUSELIGHT_W: Q6.D, X1.19
- new net HOUSELIGHT_W_GPIO: Q6.G, U1.PWM3
- new net IR_3: R24.1, R30.1, X2.23
- new net IR_3_GPIO: IC2A.O, SV1.22, SV2.22
- new net IR_4: R25.1, R31.1, X2.22
- new net IR_4_GPIO: IC2B.O, SV1.38
- new net IR_5: R26.1, R32.1, X2.21
- new net IR_5_GPIO: IC2C.O, SV1.40
- new net IR_6: R27.1, R33.1, X2.20
- new net IR_6_GPIO: IC2D.O, SV1.35, SV2.35
- new net IR_7: R28.1, R34.1
- new net IR_8: R29.1, R35.1
- new net LED_1: R38.1, X2.13
- new net LED_2: R9.1, X2.12
- new net LED_3: R10.1, X2.11
- new net LED_4: R11.1, X2.10
- new net LED_5: R12.1, X2.9
- new net LED_6: R21.1, X2.8
- new net LOADCELL2A+: X2.16
- new net LOADCELL2A-: X2.15
- new net LOADCELLA+: X1.15
- new net LOADCELLA-: X1.14
- new net LOADCELLE+: X1.25
- new net LOADCELLE-: X1.24
- new net N$11: IC2F.I, R29.2
- new net N$13: R17.2, U1.PWM4
- new net N$14: R36.2, U1.PWM5
- new net N$15: R37.2, U1.PWM6
- new net N$16: R38.2, U1.PWM7
- new net N$17: IC2E.O
- new net N$18: IC2F.O
- new net N$26: R9.2, U1.PWM8
- new net N$28: R11.2, U1.PWM10
- new net N$29: R12.2, U1.PWM11
- new net N$3: IC2A.I, R24.2
- new net N$30: R21.2, U1.PWM12
- new net N$4: IC2B.I, R25.2
- new net N$5: IC2C.I, R26.2
- new net N$7: IC2D.I, R27.2
- new net N$9: IC2E.I, R28.2
- new net RGB_CUE_B: X1.4
- new net RGB_CUE_G: X1.3
- new net RGB_CUE_R: X1.5
- new net RXD: J7.2, SV1.10
- new net SCL: SV1.5, U1.SCL
- new net SDA: SV1.3, U1.SDA
- new net TEMP: X1.2
- new net TXD: J7.1, SV1.8
- new net USB1_D+: J1.D+, X1.16
- new net USB1_D-: J1.D-, X1.17
- new net USB1_VBUS: J1.VBUS, X1.18
- new net USB2_D+: J4.D+, X2.17
- new net USB2_D-: J4.D-, X2.18
- new net USB2_VBUS: J4.VBUS, X2.19
- net +3V3: now also IC2P.VCC, R30.2, R31.2, R32.2, R33.2, R34.2, R35.2, U1.A0, U1.A2, U1.A4, U1.VDD; no longer R10.2, R11.2, R12.2, R9.2
- net +5V: no longer X1.25
- net 12V: no longer D2.C, X1.24
- net ADC0: now also X1.1; no longer X1.2
- net ADC1: now also X2.14; no longer X1.1
- net ADC2: now also X2.7; no longer X1.17
- net ADC3: now also X2.6
- net ADC4: now also X2.5; no longer X1.16
- net CENTER_LED: no longer R22.1
- net GND: now also IC2P.GND, J1.GND, J4.GND, Q3.S, Q4.S, Q5.S, Q6.S, U1.#OE, U1.A1, U1.A3, U1.A5, U1.EXTCLK, U1.GND, X2.G1, X2.G2; no longer Q2.S
- net GPIO17: now also J9.1; no longer R23.1
- net GPIO22: now also J8.2; no longer R21.1
- net GPIO27: now also J8.1; no longer R22.2
- net IR_1: now also X2.25; no longer X1.4
- net IR_2: now also X2.24; no longer X1.3
- net LEFT_LED: now also R17.1; no longer R23.2
- net N$27: now also R10.2, U1.PWM9; no longer Q2.G, R17.2
- net RIGHT_LED: now also R37.1; no longer R21.2
Other:
- moved on the sheet: R10, R11, R12, R17, R21, R9

Commit message: new board
Connections:
- net GND: now also J1.SHIELD, J4.SHIELD
Changed lines of the file:
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@@
 <?xml version="1.0" encoding="utf-8"?>
 <!DOCTYPE eagle SYSTEM "eagle.dtd">
-<eagle version="8.4.1">
+<eagle version="8.4.3">
 <drawing>
 <settings>
@@
 <part name="R12" library="resistor" library_urn="urn:adsk.eagle:library:348" deviceset="R-US_" device="0207/7" package3d_urn="urn:adsk.eagle:package:25942/1" value="330"/>
 <part name="R21" library="resistor" library_urn="urn:adsk.eagle:library:348" deviceset="R-US_" device="0207/7" package3d_urn="urn:adsk.eagle:package:25942/1" value="330"/>
+<part name="GND15" library="SparkFun-PowerSymbols" deviceset="GND" device=""/>
 </parts>
 <sheets>
@@
 <instance part="R12" gate="G$1" x="53.34" y="187.96" rot="R180"/>
 <instance part="R21" gate="G$1" x="53.34" y="180.34" rot="R180"/>
+<instance part="GND15" gate="1" x="-218.44" y="193.04"/>
 </instances>
 <busses>
@@
 <junction x="-35.56" y="233.68"/>
 </segment>
+<segment>
+<pinref part="J1" gate="G$1" pin="SHIELD"/>
+<pinref part="GND15" gate="1" pin="GND"/>
+<wire x1="-226.06" y1="182.88" x2="-226.06" y2="195.58" width="0.1524" layer="91"/>
+<wire x1="-226.06" y1="195.58" x2="-218.44" y2="195.58" width="0.1524" layer="91"/>
+<pinref part="J4" gate="G$1" pin="SHIELD"/>
+<wire x1="-218.44" y1="195.58" x2="-208.28" y2="195.58" width="0.1524" layer="91"/>
+<wire x1="-208.28" y1="195.58" x2="-208.28" y2="182.88" width="0.1524" layer="91"/>
+<junction x="-218.44" y="195.58"/>
+</segment>
 </net>
