File: RPiOperant.sch (EAGLE design)
At the start: 62 parts, among them IC1 74LS14N, IC2 74LS14N, IC3 MCP3008, J1 USB_B_PTH, J2 POWER_JACK, J3 POWER_JACK, J4 USB_B_PTH, J5 1X2-3.5MM, J6 1X2-3.5MM, J7 1X2-3.5MM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

Commit message: new stuff!
Parts:
- removed J7, J8, J9: 1X2-3.5MM, adafruit:1X2-3.5MM
- added J10, J13, J14: (no value), SparkFun-Connectors:CONN_03SCREW
- added J11, J12: (no value), SparkFun-Connectors:CONN_05
- added JP1: (no value), jumper:JP2E
- added Q2, Q7: 60V/32A/35mΩ, SparkFun-DiscreteSemi:MOSFET-NCH-FQP30N06L
- added R40, R41: 10K, resistor:R-US_0207/7
Connections:
- removed net TEMP: X1.2
- new net DAT: J12.3
- new net LCCLK: J12.2
- new net TTL27: J10.1, Q2.D, R41.2
- new net YLW: J11.1
- net +3V3: now also J12.4
- net GND: now also J10.3, J12.1, J13.3, J14.3
- net GPIO17: now also J13.1; no longer J9.1
- net GPIO18: now also J13.2, X1.2; no longer J9.2
- net GPIO22: now also J10.2; no longer J8.2
- net GPIO27: now also Q2.S, R40.2; no longer J8.1
- net LOADCELLA+: now also J11.3
- net LOADCELLA-: now also J11.2
- net LOADCELLE+: now also J11.5
- net LOADCELLE-: now also J11.4
- net RPI_3.3V: now also JP1.1, Q2.G, R40.1
- net RPI_5V: now also JP1.2, JP1.3, R41.1
- net RXD: now also J14.2; no longer J7.2
- net TXD: now also J14.1; no longer J7.1

Commit message: final draft
Parts:
- removed Q2, Q7: 60V/32A/35mΩ, SparkFun-DiscreteSemi:MOSFET-NCH-FQP30N06L
- removed R40, R41: 10K, resistor:R-US_0207/7
- added B1: SPARKFUN_LOGIC_LEVEL_CONVERTER, SparkFun-Boards:SPARKFUN_LOGIC_LEVEL_CONVERTER
- added JP2, JP3, JP4: (no value), jumper:JP2E
Connections:
- new net N$22: B1.HV_TXO_1, JP2.3
- new net N$23: B1.HV_RXI_1, JP3.3
- new net N$32: J13.1, JP1.1
- new net N$33: J13.2, JP4.1
- new net TTL22: J10.2, JP3.2
- net +3V3: now also J12.5; no longer J12.4
- net +5V: now also J12.4
- net DAT: now also JP1.3
- net GND: now also B1.GND, B1.GND@2
- net GPIO17: now also JP1.2; no longer J13.1
- net GPIO18: now also JP4.2; no longer J13.2
- net GPIO22: now also B1.LV_RXO_1, JP3.1; no longer J10.2
- net GPIO27: now also B1.LV_TXI_1, JP2.1; no longer Q2.S, R40.2
- net LCCLK: now also JP4.3
- net RPI_3.3V: now also B1.LV; no longer JP1.1, Q2.G, R40.1
- net RPI_5V: now also B1.HV; no longer JP1.2, JP1.3, R41.1
- net TTL27: now also JP2.2; no longer Q2.D, R41.2
Other:
- moved on the sheet: JP1

Commit message: alternate
Parts:
- removed IC3: MCP3008, adafruit:MCP3008
- removed J1, J4: USB_B_PTH, SparkFun-Connectors:USB_B_PTH
- removed J5, J6: 1X2-3.5MM, adafruit:1X2-3.5MM
- added J15, J9: (no value), SparkFun-Connectors:CONN_023.5MM
- added J7, J8: (no value), SparkFun-Connectors:CONN_04
Connections:
- removed net ADC0: IC3.CH0, X1.1
- removed net ADC1: IC3.CH1, X2.14
- removed net ADC2: IC3.CH2, X2.7
- removed net ADC3: IC3.CH3, X2.6
- removed net ADC4: IC3.CH4, X2.5
- removed net ADC5: IC3.CH5
- removed net ADC6: IC3.CH6
- removed net ADC7: IC3.CH7
- removed net CE0: SV1.24, SV2.24
- removed net CE1: IC3./CS, SV1.26, SV2.26
- removed net GPIO18: JP4.2, SV1.12, X1.2
- removed net MISO: IC3.DOUT, SV1.21, SV2.21
- removed net MOSI: IC3.DIN, SV1.19, SV2.19
- removed net SCLK: IC3.CLK, SV1.23, SV2.23
- new net GPIO7: SV1.26, SV2.26
- new net GPIO8: JP4.2, SV1.24, SV2.24
- new net N$25: X2.7
- new net N$31: X2.6
- new net N$34: X2.5
- new net N$35: X2.14
- net +3V3: no longer IC3.VDD, IC3.VREF
- net AUX1: now also J9.1; no longer J5.1, SV1.7
- net AUX2: now also J9.2; no longer J5.2
- net AUX3: now also J15.1; no longer J6.1
- net AUX4: now also J15.2; no longer J6.2
- net GND: now also J7.4, J8.4; no longer IC3.AGND, IC3.GND, J1.GND, J1.SHIELD, J4.GND, J4.SHIELD
- net IR_4_GPIO: now also SV1.21, SV2.21; no longer SV1.38
- net IR_5_GPIO: now also SV1.23, SV2.23; no longer SV1.40
- net IR_6_GPIO: now also SV1.19, SV2.19; no longer SV1.35, SV2.35
- net TTL22: now also X1.2
- net TTL27: now also X1.1
- net USB1_D+: now also J7.3; no longer J1.D+
- net USB1_D-: now also J7.2; no longer J1.D-
- net USB1_VBUS: now also J7.1; no longer J1.VBUS
- net USB2_D+: now also J8.3; no longer J4.D+
- net USB2_D-: now also J8.2; no longer J4.D-
- net USB2_VBUS: now also J8.1; no longer J4.VBUS

Commit message: final draft
Parts:
- added J1: (no value), SparkFun-Connectors:CONN_04SCREW
Connections:
- removed net N$25: X2.7
- removed net N$31: X2.6
- removed net N$34: X2.5
- removed net N$35: X2.14
- new net AUX5: J1.1, X2.5
- new net AUX6: J1.2, X2.6
- new net AUX7: J1.3, X2.7
- new net AUX8: J1.4, X2.14
Changed lines of the file:
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@@
 <part name="J9" library="SparkFun-Connectors" deviceset="CONN_02" device="3.5MM"/>
 <part name="J15" library="SparkFun-Connectors" deviceset="CONN_02" device="3.5MM"/>
+<part name="J1" library="SparkFun-Connectors" deviceset="CONN_04" device="SCREW"/>
 </parts>
 <sheets>
@@
 <instance part="J9" gate="G$1" x="-175.26" y="226.06" rot="R180"/>
 <instance part="J15" gate="G$1" x="-175.26" y="213.36" rot="R180"/>
+<instance part="J1" gate="G$1" x="-139.7" y="208.28" rot="R270"/>
 </instances>
 <busses>
@@
 </segment>
 </net>
-<net name="N$25" class="0">
+<net name="AUX5" class="0">
+<segment>
+<pinref part="J1" gate="G$1" pin="1"/>
+<wire x1="-142.24" y1="203.2" x2="-142.24" y2="190.5" width="0.1524" layer="91"/>
+<label x="-142.24" y="190.5" size="1.27" layer="91" rot="R270" xref="yes"/>
+</segment>
+<segment>
+<pinref part="X2" gate="G$1" pin="5"/>
+<wire x1="-152.4" y1="144.78" x2="-152.4" y2="152.4" width="0.1524" layer="91"/>
+<label x="-152.4" y="152.4" size="1.27" layer="91" rot="R90" xref="yes"/>
+</segment>
+</net>
+<net name="AUX6" class="0">
+<segment>
+<pinref part="J1" gate="G$1" pin="2"/>
+<wire x1="-139.7" y1="203.2" x2="-139.7" y2="190.5" width="0.1524" layer="91"/>
+<label x="-139.7" y="190.5" size="1.27" layer="91" rot="R270" xref="yes"/>
+</segment>
+<segment>
+<pinref part="X2" gate="G$1" pin="6"/>
+<wire x1="-154.94" y1="144.78" x2="-154.94" y2="152.4" width="0.1524" layer="91"/>
+<label x="-154.94" y="152.4" size="1.27" layer="91" rot="R90" xref="yes"/>
+</segment>
+</net>
+<net name="AUX7" class="0">
+<segment>
+<pinref part="J1" gate="G$1" pin="3"/>
+<wire x1="-137.16" y1="203.2" x2="-137.16" y2="190.5" width="0.1524" layer="91"/>
+<label x="-137.16" y="190.5" size="1.27" layer="91" rot="R270" xref="yes"/>
+</segment>
 <segment>
 <pinref part="X2" gate="G$1" pin="7"/>
@@
 </segment>
 </net>
-<net name="N$31" class="0">
-<segment>
-<pinref part="X2" gate="G$1" pin="6"/>
-<wire x1="-154.94" y1="144.78" x2="-154.94" y2="152.4" width="0.1524" layer="91"/>
-<label x="-154.94" y="152.4" size="1.27" layer="91" rot="R90" xref="yes"/>
-</segment>
-</net>
-<net name="N$34" class="0">
-<segment>
-<pinref part="X2" gate="G$1" pin="5"/>
-<wire x1="-152.4" y1="144.78" x2="-152.4" y2="152.4" width="0.1524" layer="91"/>
-<label x="-152.4" y="152.4" size="1.27" layer="91" rot="R90" xref="yes"/>
-</segment>
-</net>
-<net name="N$35" class="0">
+<net name="AUX8" class="0">
+<segment>
+<pinref part="J1" gate="G$1" pin="4"/>
+<wire x1="-134.62" y1="203.2" x2="-134.62" y2="190.5" width="0.1524" layer="91"/>
+<label x="-134.62" y="190.5" size="1.27" layer="91" rot="R270" xref="yes"/>
+</segment>
 <segment>
 <pinref part="X2" gate="G$1" pin="14"/>

Commit message: revision b
Parts:
- removed SV2: (no value), con-lstb:MA20-2
- added SV3: (no value), con-lstb:MA20-2
Connections:
- removed net CENTNER_IR: R5.1, R6.1
- new net GPIO4: SV1.7, SV3.7
- new net ID_SC: SV1.28, SV3.28
- new net ID_SD: SV1.27, SV3.27
- new net PCM_CLK: SV1.12, SV3.12
- new net PCM_DIN: SV1.38, SV3.38
- new net PCM_DOUT: SV1.40, SV3.40
- new net PCM_FS: SV1.35, SV3.35
- net AUX2: now also SV3.32
- net CENTER_IR: now also R5.1, R6.1
- net CENTER_PECK_GPIO: now also SV3.33; no longer SV2.33
- net GND: now also SV3.14, SV3.20, SV3.25, SV3.30, SV3.34, SV3.39, SV3.6, SV3.9; no longer SV2.14, SV2.20, SV2.25, SV2.30, SV2.34, SV2.39, SV2.6, SV2.9
- net GPIO17: now also SV3.11; no longer SV2.11
- net GPIO22: now also SV3.15; no longer SV2.15
- net GPIO27: now also SV3.13; no longer SV2.13
- net GPIO7: now also SV3.26; no longer SV2.26
- net GPIO8: now also SV3.24; no longer SV2.24
- net HOPPER_IR_GPIO: now also SV3.29; no longer SV2.29
- net HOPPER_TRIG_GPIO: now also SV3.36; no longer SV2.36
- net IR_1_GPIO: now also SV3.16
- net IR_2_GPIO: now also SV3.18; no longer SV2.18
- net IR_3_GPIO: now also SV3.22; no longer SV2.22
- net IR_4_GPIO: now also SV3.21; no longer SV2.21
- net IR_5_GPIO: now also SV3.23; no longer SV2.23
- net IR_6_GPIO: now also SV3.19; no longer SV2.19
- net LEFT_PECK_GPIO: now also SV3.31; no longer SV2.31
- net RIGHT_PECK_GPIO: now also SV3.37; no longer SV2.37
- net RPI_3.3V: now also SV3.1, SV3.17; no longer SV2.1, SV2.17
- net RPI_5V: now also SV3.2, SV3.4; no longer SV2.2, SV2.4
- net RXD: now also SV3.10
- net SCL: now also SV3.5
- net SDA: now also SV3.3
- net TXD: now also SV3.8

Commit message: updates
Parts:
- removed J3: POWER_JACK, SparkFun-Connectors:POWER_JACK
- removed R18: 10k, resistor:R-US_0207/7
- removed R19: 20k, resistor:R-US_0207/7
- added C1: 100nF, adafruit:C-US050-025X075
- added C2, C3, C4: 10uF, adafruit:C-US050-025X075
- added U$1: V_REG_LD1117VXX, SparkFun-IC-Power:V_REG_LD1117VXX
- added U2: (no value), SparkFun-IC-Power:V_REG_78XX-TO-220
Connections:
- new net 5V: C4.1, U2.OUT
- net +3V3: now also C2.1, U$1.OUT; no longer R18.1, R19.2
- net +5V: no longer J3.PWR, R18.2
- net 12V: now also C1.1, C3.1, U$1.IN, U2.IN
- net GND: now also C1.2, C2.2, C3.2, C4.2, U$1.GND, U2.GND; no longer J3.GND, J3.GNDBREAK, R19.1

Commit message: version 2
Parts:
- removed C3, C4: 10uF, adafruit:C-US050-025X075
- removed U2: (no value), SparkFun-IC-Power:V_REG_78XX-TO-220
Connections:
- removed net 5V: C4.1, U2.OUT
- net 12V: now also X1.23; no longer C3.1, U2.IN
- net GND: no longer C3.2, C4.2, U2.GND, X1.23
Changed lines of the file:
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@@
 <part name="C1" library="adafruit" deviceset="C-US" device="050-025X075" value="100nF"/>
 <part name="C2" library="adafruit" deviceset="C-US" device="050-025X075" value="10uF"/>
-<part name="U2" library="SparkFun-IC-Power" library_urn="urn:adsk.eagle:library:526" deviceset="V_REG_78XX" device="-TO-220" package3d_urn="urn:adsk.eagle:package:39066/1"/>
 <part name="SUPPLY1" library="SparkFun-PowerSymbols" deviceset="12V" device=""/>
-<part name="SUPPLY3" library="SparkFun-PowerSymbols" deviceset="12V" device=""/>
-<part name="C3" library="adafruit" deviceset="C-US" device="050-025X075" value="10uF"/>
-<part name="C4" library="adafruit" deviceset="C-US" device="050-025X075" value="10uF"/>
-<part name="GND6" library="SparkFun-PowerSymbols" deviceset="GND" device=""/>
-<part name="SUPPLY4" library="SparkFun-PowerSymbols" library_urn="urn:adsk.eagle:library:530" deviceset="5V" device=""/>
 </parts>
 <sheets>
@@
 <instance part="C1" gate="G$1" x="17.78" y="124.46"/>
 <instance part="C2" gate="G$1" x="55.88" y="124.46"/>
-<instance part="U2" gate="G$1" x="86.36" y="137.16"/>
 <instance part="SUPPLY1" gate="G$1" x="17.78" y="144.78"/>
-<instance part="SUPPLY3" gate="G$1" x="71.12" y="144.78"/>
-<instance part="C3" gate="G$1" x="71.12" y="124.46"/>
-<instance part="C4" gate="G$1" x="99.06" y="124.46"/>
-<instance part="GND6" gate="1" x="86.36" y="111.76"/>
-<instance part="SUPPLY4" gate="G$1" x="99.06" y="144.78"/>
 </instances>
 <busses>
@@
 <wire x1="-88.9" y1="129.54" x2="-88.9" y2="121.92" width="0.1524" layer="91"/>
 <label x="-88.9" y="121.92" size="1.016" layer="91" rot="R270" xref="yes"/>
-</segment>
-<segment>
-<pinref part="X1" gate="G$1" pin="23"/>
-<wire x1="-114.3" y1="129.54" x2="-114.3" y2="121.92" width="0.1524" layer="91"/>
-<label x="-114.3" y="121.92" size="1.016" layer="91" rot="R270" xref="yes"/>
 </segment>
 <segment>
@@
 <wire x1="33.02" y1="129.54" x2="33.02" y2="119.38" width="0.1524" layer="91"/>
 </segment>
-<segment>
-<pinref part="C3" gate="G$1" pin="2"/>
-<pinref part="GND6" gate="1" pin="GND"/>
-<wire x1="71.12" y1="119.38" x2="71.12" y2="114.3" width="0.1524" layer="91"/>
-<wire x1="71.12" y1="114.3" x2="86.36" y2="114.3" width="0.1524" layer="91"/>
-<pinref part="C4" gate="G$1" pin="2"/>
-<wire x1="86.36" y1="114.3" x2="99.06" y2="114.3" width="0.1524" layer="91"/>
-<wire x1="99.06" y1="114.3" x2="99.06" y2="119.38" width="0.1524" layer="91"/>
-<junction x="86.36" y="114.3"/>
-<pinref part="U2" gate="G$1" pin="GND"/>
-<wire x1="86.36" y1="129.54" x2="86.36" y2="114.3" width="0.1524" layer="91"/>
-</segment>
 </net>
 <net name="12V" class="1">
@@
 </segment>
 <segment>
-<pinref part="C3" gate="G$1" pin="1"/>
-<pinref part="SUPPLY3" gate="G$1" pin="12V"/>
-<wire x1="71.12" y1="127" x2="71.12" y2="137.16" width="0.1524" layer="91"/>
-<pinref part="U2" gate="G$1" pin="IN"/>
-<wire x1="71.12" y1="137.16" x2="71.12" y2="144.78" width="0.1524" layer="91"/>
-<wire x1="78.74" y1="137.16" x2="71.12" y2="137.16" width="0.1524" layer="91"/>
-<junction x="71.12" y="137.16"/>
+<pinref part="X1" gate="G$1" pin="23"/>
+<wire x1="-114.3" y1="129.54" x2="-114.3" y2="121.92" width="0.1524" layer="91"/>
+<label x="-114.3" y="121.92" size="0.8128" layer="91" rot="R270" xref="yes"/>
 </segment>
 </net>
@@
 </segment>
 </net>
-<net name="5V" class="0">
-<segment>
-<pinref part="U2" gate="G$1" pin="OUT"/>
-<pinref part="C4" gate="G$1" pin="1"/>
-<wire x1="93.98" y1="137.16" x2="99.06" y2="137.16" width="0.1524" layer="91"/>
-<wire x1="99.06" y1="137.16" x2="99.06" y2="127" width="0.1524" layer="91"/>
-<wire x1="99.06" y1="137.16" x2="99.06" y2="144.78" width="0.1524" layer="91"/>
-<junction x="99.06" y="137.16"/>
-<pinref part="SUPPLY4" gate="G$1" pin="5V"/>
-</segment>
-</net>
