File: RPiOperant.sch (EAGLE design)
At the start: 66 parts, among them IC1 74LS14N, IC2 74LS14N, J2 POWER_JACK, X1 2516-, X2 22-23-2041, X3 2550-

Commit message: rev_c v1
Parts:
- added C1: 100nF, adafruit:C-US050-025X075
- added C2: 10uF, adafruit:C-US050-025X075
- added U3: (no value), SparkFun-IC-Power:V_REG_78XXSINK
Connections:
- new net 24V: C1.1, C3.1, J2.PWR, U2.IN, U3.IN, X3-1.KL
- net 12V: now also C2.1, U3.OUT; no longer C3.1, J2.PWR, U2.IN, X3-1.KL
- net GND: now also C1.2, C2.2, U3.GND
Changed lines of the file:
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@@
 <part name="J2" library="SparkFun-Connectors" deviceset="POWER_JACK" device=""/>
 <part name="GND1" library="SparkFun-PowerSymbols" deviceset="GND" device=""/>
-<part name="SUPPLY2" library="SparkFun-PowerSymbols" deviceset="12V" device=""/>
 <part name="IC1" library="74xx-us" library_urn="urn:adsk.eagle:library:88" deviceset="74*14" device="N" package3d_urn="urn:adsk.eagle:package:2921/1" technology="LS">
 <attribute name="SPICEPREFIX" value="I"/>
@@
 <part name="GND6" library="SparkFun-PowerSymbols" deviceset="GND" device=""/>
 <part name="+3V1" library="supply1" library_urn="urn:adsk.eagle:library:371" deviceset="+3V3" device=""/>
-<part name="SUPPLY3" library="SparkFun-PowerSymbols" deviceset="12V" device=""/>
 <part name="X3" library="con-3m" library_urn="urn:adsk.eagle:library:119" deviceset="2550-" device="" package3d_urn="urn:adsk.eagle:package:5594/1"/>
 <part name="X1" library="con-3m" library_urn="urn:adsk.eagle:library:119" deviceset="2516-" device="" package3d_urn="urn:adsk.eagle:package:5574/1"/>
@@
 <part name="R18" library="resistor" library_urn="urn:adsk.eagle:library:348" deviceset="R-US_" device="0207/7" package3d_urn="urn:adsk.eagle:package:25942/1" value="330"/>
 <part name="R19" library="resistor" library_urn="urn:adsk.eagle:library:348" deviceset="R-US_" device="0207/7" package3d_urn="urn:adsk.eagle:package:25942/1" value="330"/>
+<part name="U3" library="SparkFun-IC-Power" deviceset="V_REG_78XX" device="SINK"/>
+<part name="GND12" library="SparkFun-PowerSymbols" deviceset="GND" device=""/>
+<part name="C1" library="adafruit" deviceset="C-US" device="050-025X075" value="100nF"/>
+<part name="C2" library="adafruit" deviceset="C-US" device="050-025X075" value="10uF"/>
 </parts>
 <sheets>
@@
 <instance part="J2" gate="G$1" x="-12.7" y="116.84"/>
 <instance part="GND1" gate="1" x="-2.54" y="111.76"/>
-<instance part="SUPPLY2" gate="G$1" x="2.54" y="127"/>
 <instance part="IC1" gate="A" x="-134.62" y="78.74"/>
 <instance part="IC1" gate="B" x="-134.62" y="38.1"/>
@@
 <instance part="GND6" gate="1" x="-30.48" y="137.16"/>
 <instance part="+3V1" gate="G$1" x="-17.78" y="175.26"/>
-<instance part="SUPPLY3" gate="G$1" x="-43.18" y="172.72"/>
 <instance part="X3" gate="-1" x="-231.14" y="162.56"/>
 <instance part="X3" gate="-2" x="-205.74" y="162.56"/>
@@
 <instance part="R18" gate="G$1" x="-119.38" y="162.56" rot="R180"/>
 <instance part="R19" gate="G$1" x="-119.38" y="170.18" rot="R180"/>
+<instance part="U3" gate="G$1" x="-60.96" y="124.46"/>
+<instance part="GND12" gate="1" x="-60.96" y="106.68"/>
+<instance part="C1" gate="G$1" x="-76.2" y="114.3"/>
+<instance part="C2" gate="G$1" x="-45.72" y="114.3"/>
 </instances>
 <busses>
@@
 <junction x="-101.6" y="160.02"/>
 </segment>
+<segment>
+<pinref part="U3" gate="G$1" pin="GND"/>
+<pinref part="GND12" gate="1" pin="GND"/>
+<wire x1="-60.96" y1="116.84" x2="-60.96" y2="109.22" width="0.1524" layer="91"/>
+<pinref part="C1" gate="G$1" pin="2"/>
+<wire x1="-76.2" y1="109.22" x2="-60.96" y2="109.22" width="0.1524" layer="91"/>
+<pinref part="C2" gate="G$1" pin="2"/>
+<wire x1="-60.96" y1="109.22" x2="-45.72" y2="109.22" width="0.1524" layer="91"/>
+</segment>
 </net>
 <net name="12V" class="1">
-<segment>
-<pinref part="J2" gate="G$1" pin="PWR"/>
-<wire x1="-10.16" y1="124.46" x2="2.54" y2="124.46" width="0.1524" layer="91"/>
-<pinref part="SUPPLY2" gate="G$1" pin="12V"/>
-<wire x1="2.54" y1="124.46" x2="2.54" y2="127" width="0.1524" layer="91"/>
-</segment>
 <segment>
 <pinref part="SUPPLY11" gate="G$1" pin="12V"/>
@@
 </segment>
 <segment>
-<pinref part="C3" gate="G$1" pin="1"/>
-<pinref part="U2" gate="G$1" pin="IN"/>
-<wire x1="-43.18" y1="152.4" x2="-43.18" y2="165.1" width="0.1524" layer="91"/>
-<wire x1="-43.18" y1="165.1" x2="-38.1" y2="165.1" width="0.1524" layer="91"/>
-<pinref part="SUPPLY3" gate="G$1" pin="12V"/>
-<wire x1="-43.18" y1="165.1" x2="-43.18" y2="172.72" width="0.1524" layer="91"/>
-<junction x="-43.18" y="165.1"/>
-</segment>
-<segment>
-<pinref part="X3" gate="-1" pin="KL"/>
-<wire x1="-226.06" y1="162.56" x2="-223.52" y2="162.56" width="0.1524" layer="91"/>
-<label x="-223.52" y="162.56" size="1.27" layer="91" xref="yes"/>
-</segment>
-<segment>
 <pinref part="X3" gate="-23" pin="KL"/>
 <wire x1="-226.06" y1="134.62" x2="-223.52" y2="134.62" width="0.1524" layer="91"/>
 <label x="-223.52" y="134.62" size="1.27" layer="91" xref="yes"/>
+</segment>
+<segment>
+<label x="-45.72" y="132.08" size="1.778" layer="91" rot="R90" xref="yes"/>
+<pinref part="C2" gate="G$1" pin="1"/>
+<wire x1="-45.72" y1="116.84" x2="-45.72" y2="124.46" width="0.1524" layer="91"/>
+<pinref part="U3" gate="G$1" pin="OUT"/>
+<wire x1="-45.72" y1="124.46" x2="-45.72" y2="132.08" width="0.1524" layer="91"/>
+<wire x1="-53.34" y1="124.46" x2="-45.72" y2="124.46" width="0.1524" layer="91"/>
 </segment>
 </net>
@@
 </segment>
 </net>
+<net name="24V" class="1">
+<segment>
+<pinref part="C3" gate="G$1" pin="1"/>
+<pinref part="U2" gate="G$1" pin="IN"/>
+<wire x1="-43.18" y1="152.4" x2="-43.18" y2="165.1" width="0.1524" layer="91"/>
+<wire x1="-43.18" y1="165.1" x2="-38.1" y2="165.1" width="0.1524" layer="91"/>
+<wire x1="-43.18" y1="165.1" x2="-43.18" y2="172.72" width="0.1524" layer="91"/>
+<junction x="-43.18" y="165.1"/>
+<label x="-43.18" y="172.72" size="1.778" layer="91" rot="R90" xref="yes"/>
+</segment>
+<segment>
+<pinref part="J2" gate="G$1" pin="PWR"/>
+<wire x1="-10.16" y1="124.46" x2="2.54" y2="124.46" width="0.1524" layer="91"/>
+<wire x1="2.54" y1="124.46" x2="2.54" y2="127" width="0.1524" layer="91"/>
+<label x="2.54" y="127" size="1.778" layer="91" rot="R90" xref="yes"/>
+</segment>
+<segment>
+<wire x1="-76.2" y1="116.84" x2="-76.2" y2="124.46" width="0.1524" layer="91"/>
+<label x="-76.2" y="134.62" size="1.778" layer="91" rot="R90" xref="yes"/>
+<pinref part="C1" gate="G$1" pin="1"/>
+<pinref part="U3" gate="G$1" pin="IN"/>
+<wire x1="-76.2" y1="124.46" x2="-76.2" y2="134.62" width="0.1524" layer="91"/>
+<wire x1="-76.2" y1="124.46" x2="-68.58" y2="124.46" width="0.1524" layer="91"/>
+</segment>
+<segment>
+<pinref part="X3" gate="-1" pin="KL"/>
+<wire x1="-226.06" y1="162.56" x2="-223.52" y2="162.56" width="0.1524" layer="91"/>
+<label x="-223.52" y="162.56" size="1.778" layer="91" xref="yes"/>
+</segment>
+</net>

Commit message: rev c updates
Parts:
- removed J7, J8: (no value), SparkFun-Connectors:CONN_04
- added X4: (no value), con-subd:F15H
- J2: value POWER_JACK -> (none); device SparkFun-Connectors:POWER_JACK -> InputOutputIO (rev18a):61400826021
- X1: value 2516- -> (none); device con-3m:2516- -> con-molex:KK-156-2
Connections:
- net +3V3: now also X4.8
- net 12V: no longer D1.C
- net 24V: now also D1.C, X1-1.S; no longer J2.PWR
- net AUX1: now also X4.7; no longer X1-1.KL
- net AUX2: now also X4.6; no longer X1-2.KL
- net AUX3: now also X4.5; no longer X1-3.KL
- net AUX4: now also X4.4; no longer X1-4.KL
- net AUX5: now also X4.3; no longer X1-5.KL
- net AUX6: now also X4.2; no longer X1-6.KL
- net AUX7: no longer X1-7.KL
- net AUX8: now also X4.1; no longer X1-8.KL
- net GND: now also J2.A_GND, J2.A_SHIELD, J2.B_GND, J2.B_SHIELD, X1-2.S, X4.9; no longer J2.GND, J2.GNDBREAK, J7.4, J8.4, X1-15.KL, X1-16.KL
- net GPIO17EXT: now also X4.15; no longer X1-9.KL
- net GPIO8EXT: now also X4.14; no longer X1-10.KL
- net RXD: now also X4.10; no longer X1-14.KL
- net TTL22: now also X4.12; no longer X1-12.KL
- net TTL27: now also X4.13; no longer X1-11.KL
- net TXD: now also X4.11; no longer X1-13.KL
- net USB1_D+: now also J2.A_D+; no longer J7.3
- net USB1_D-: now also J2.A_D-; no longer J7.2
- net USB1_VBUS: now also J2.A_VBUS; no longer J7.1
- net USB2_D+: now also J2.B_D+; no longer J8.3
- net USB2_D-: now also J2.B_D-; no longer J8.2
- net USB2_VBUS: now also J2.B_VBUS; no longer J8.1
Other:
- moved on the sheet: X1-1, X1-2

Commit message: revision C
Parts:
- added U$1: HDMI-A, connectors:HDMI-A
Connections:
- net +3V3: now also X3-23.KL; no longer X3-2.KL
- net 12V: now also X3-2.KL; no longer X3-23.KL
- net CENTER_PECK_GPIO: now also U$1.DATA0-
- net GND: now also U$1.CEC, U$1.CECGND, U$1.CLOCKSHIELD, U$1.DATA0SHIELD, U$1.DATA1SHIELD, U$1.DATA2SHIELD, U$1.HOTPLUG, U$1.SCL, U$1.SDA, U$1.UTIL, U$1.VCC
- net HOPPER_TRIG_GPIO: now also U$1.CLOCK-
- net LEFT_PECK_GPIO: now also U$1.DATA0+
- net RIGHT_PECK_GPIO: now also U$1.CLOCK+
- net RXD: now also U$1.DATA2-
- net TTL22: now also U$1.DATA1-
- net TTL27: now also U$1.DATA1+
- net TXD: now also U$1.DATA2+
Changed lines of the file:
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@@
 </variantdefs>
 <classes>
-<class number="0" name="default" width="0.2032" drill="0">
+<class number="0" name="default" width="0.1524" drill="0">
 </class>
 <class number="1" name="12V" width="1.3716" drill="0">
@@
 <class number="2" name="5V" width="0.508" drill="0">
 </class>
-<class number="3" name="GND" width="0.254" drill="0">
+<class number="3" name="GND" width="0.2032" drill="0">
 </class>
 <class number="4" name="24V" width="1.3716" drill="0">
@@
 <part name="X1" library="con-molex" library_urn="urn:adsk.eagle:library:165" deviceset="KK-156-2" device=""/>
 <part name="J2" library="InputOutputIO (rev18a)" deviceset="61400826021" device=""/>
+<part name="U$1" library="connectors" deviceset="HDMI-A" device=""/>
+<part name="GND1" library="SparkFun-PowerSymbols" deviceset="GND" device=""/>
 </parts>
 <sheets>
@@
 <instance part="X1" gate="-2" x="20.32" y="116.84"/>
 <instance part="J2" gate="G$1" x="-259.08" y="218.44"/>
+<instance part="U$1" gate="G$1" x="213.36" y="20.32"/>
+<instance part="GND1" gate="1" x="226.06" y="-12.7"/>
 </instances>
 <busses>
@@
 <label x="-271.78" y="215.9" size="1.016" layer="91" rot="R90" xref="yes"/>
 </segment>
+<segment>
+<pinref part="U$1" gate="G$1" pin="UTIL"/>
+<pinref part="GND1" gate="1" pin="GND"/>
+<wire x1="218.44" y1="20.32" x2="226.06" y2="20.32" width="0.1524" layer="91"/>
+<wire x1="226.06" y1="20.32" x2="226.06" y2="17.78" width="0.1524" layer="91"/>
+<pinref part="U$1" gate="G$1" pin="HOTPLUG"/>
+<wire x1="226.06" y1="17.78" x2="226.06" y2="15.24" width="0.1524" layer="91"/>
+<wire x1="226.06" y1="15.24" x2="226.06" y2="12.7" width="0.1524" layer="91"/>
+<wire x1="226.06" y1="12.7" x2="226.06" y2="10.16" width="0.1524" layer="91"/>
+<wire x1="226.06" y1="10.16" x2="226.06" y2="7.62" width="0.1524" layer="91"/>
+<wire x1="226.06" y1="7.62" x2="226.06" y2="5.08" width="0.1524" layer="91"/>
+<wire x1="226.06" y1="5.08" x2="226.06" y2="2.54" width="0.1524" layer="91"/>
+<wire x1="226.06" y1="2.54" x2="226.06" y2="0" width="0.1524" layer="91"/>
+<wire x1="226.06" y1="0" x2="226.06" y2="-2.54" width="0.1524" layer="91"/>
+<wire x1="226.06" y1="-2.54" x2="226.06" y2="-5.08" width="0.1524" layer="91"/>
+<wire x1="226.06" y1="-5.08" x2="226.06" y2="-10.16" width="0.1524" layer="91"/>
+<wire x1="218.44" y1="17.78" x2="226.06" y2="17.78" width="0.1524" layer="91"/>
+<junction x="226.06" y="17.78"/>
+<pinref part="U$1" gate="G$1" pin="SDA"/>
+<wire x1="218.44" y1="15.24" x2="226.06" y2="15.24" width="0.1524" layer="91"/>
+<junction x="226.06" y="15.24"/>
+<pinref part="U$1" gate="G$1" pin="SCL"/>
+<wire x1="218.44" y1="12.7" x2="226.06" y2="12.7" width="0.1524" layer="91"/>
+<junction x="226.06" y="12.7"/>
+<pinref part="U$1" gate="G$1" pin="CEC"/>
+<wire x1="218.44" y1="10.16" x2="226.06" y2="10.16" width="0.1524" layer="91"/>
+<junction x="226.06" y="10.16"/>
+<pinref part="U$1" gate="G$1" pin="VCC"/>
+<wire x1="218.44" y1="7.62" x2="226.06" y2="7.62" width="0.1524" layer="91"/>
+<junction x="226.06" y="7.62"/>
+<pinref part="U$1" gate="G$1" pin="DATA2SHIELD"/>
+<wire x1="218.44" y1="5.08" x2="226.06" y2="5.08" width="0.1524" layer="91"/>
+<junction x="226.06" y="5.08"/>
+<pinref part="U$1" gate="G$1" pin="DATA1SHIELD"/>
+<wire x1="218.44" y1="2.54" x2="226.06" y2="2.54" width="0.1524" layer="91"/>
+<junction x="226.06" y="2.54"/>
+<pinref part="U$1" gate="G$1" pin="DATA0SHIELD"/>
+<wire x1="218.44" y1="0" x2="226.06" y2="0" width="0.1524" layer="91"/>
+<junction x="226.06" y="0"/>
+<pinref part="U$1" gate="G$1" pin="CLOCKSHIELD"/>
+<wire x1="218.44" y1="-2.54" x2="226.06" y2="-2.54" width="0.1524" layer="91"/>
+<junction x="226.06" y="-2.54"/>
+<pinref part="U$1" gate="G$1" pin="CECGND"/>
+<wire x1="218.44" y1="-5.08" x2="226.06" y2="-5.08" width="0.1524" layer="91"/>
+<junction x="226.06" y="-5.08"/>
+</segment>
 </net>
 <net name="12V" class="1">
-<segment>
-<pinref part="X3" gate="-23" pin="KL"/>
-<wire x1="-226.06" y1="134.62" x2="-223.52" y2="134.62" width="0.1524" layer="91"/>
-<label x="-223.52" y="134.62" size="1.27" layer="91" xref="yes"/>
-</segment>
 <segment>
 <label x="-45.72" y="132.08" size="1.778" layer="91" rot="R90" xref="yes"/>
@@
 <wire x1="-45.72" y1="124.46" x2="-45.72" y2="132.08" width="0.1524" layer="91"/>
 <wire x1="-53.34" y1="124.46" x2="-45.72" y2="124.46" width="0.1524" layer="91"/>
+</segment>
+<segment>
+<pinref part="X3" gate="-2" pin="KL"/>
+<wire x1="-200.66" y1="162.56" x2="-198.12" y2="162.56" width="0.1524" layer="91"/>
+<label x="-198.12" y="162.56" size="1.778" layer="91" xref="yes"/>
 </segment>
 </net>
@@
 </segment>
 <segment>
-<pinref part="X3" gate="-2" pin="KL"/>
-<wire x1="-200.66" y1="162.56" x2="-198.12" y2="162.56" width="0.1524" layer="91"/>
-<label x="-198.12" y="162.56" size="1.27" layer="91" xref="yes"/>
-</segment>
-<segment>
 <pinref part="+3V7" gate="G$1" pin="+3V3"/>
 <wire x1="-127" y1="180.34" x2="-127" y2="170.18" width="0.1524" layer="91"/>
@@
 <label x="218.44" y="73.66" size="1.778" layer="91" xref="yes"/>
 </segment>
+<segment>
+<pinref part="X3" gate="-23" pin="KL"/>
+<wire x1="-226.06" y1="134.62" x2="-223.52" y2="134.62" width="0.1524" layer="91"/>
+<label x="-223.52" y="134.62" size="1.778" layer="91" xref="yes"/>
+</segment>
 </net>
 <net name="HOPPER_IR_GPIO" class="0">
@@
 <label x="-58.42" y="48.26" size="1.016" layer="91" rot="R180" xref="yes"/>
 </segment>
+<segment>
+<pinref part="U$1" gate="G$1" pin="DATA0+"/>
+<wire x1="218.44" y1="30.48" x2="231.14" y2="30.48" width="0.1524" layer="91"/>
+<label x="231.14" y="30.48" size="1.778" layer="91" xref="yes"/>
+</segment>
 </net>
 <net name="CENTER_PECK_GPIO" class="0">
@@
 <label x="-58.42" y="45.72" size="1.016" layer="91" rot="R180" xref="yes"/>
 </segment>
+<segment>
+<pinref part="U$1" gate="G$1" pin="DATA0-"/>
+<wire x1="218.44" y1="27.94" x2="231.14" y2="27.94" width="0.1524" layer="91"/>
+<label x="231.14" y="27.94" size="1.778" layer="91" xref="yes"/>
+</segment>
 </net>
 <net name="RIGHT_PECK_GPIO" class="0">
@@
 <label x="-58.42" y="40.64" size="1.016" layer="91" rot="R180" xref="yes"/>
 </segment>
+<segment>
+<pinref part="U$1" gate="G$1" pin="CLOCK+"/>
+<wire x1="218.44" y1="25.4" x2="231.14" y2="25.4" width="0.1524" layer="91"/>
+<label x="231.14" y="25.4" size="1.778" layer="91" xref="yes"/>
+</segment>
 </net>
 <net name="HOPPER_TRIG_GPIO" class="0">
@@
 <wire x1="-33.02" y1="43.18" x2="-25.4" y2="43.18" width="0.1524" layer="91"/>
 <label x="-25.4" y="43.18" size="1.016" layer="91" xref="yes"/>
+</segment>
+<segment>
+<pinref part="U$1" gate="G$1" pin="CLOCK-"/>
+<wire x1="218.44" y1="22.86" x2="231.14" y2="22.86" width="0.1524" layer="91"/>
+<label x="231.14" y="22.86" size="1.778" layer="91" xref="yes"/>
 </segment>
 </net>
@@
 <label x="193.04" y="60.96" size="1.778" layer="91" rot="R180" xref="yes"/>
 </segment>
+<segment>
+<pinref part="U$1" gate="G$1" pin="DATA2+"/>
+<wire x1="218.44" y1="40.64" x2="228.6" y2="40.64" width="0.1524" layer="91"/>
+<label x="228.6" y="40.64" size="1.778" layer="91" xref="yes"/>
+</segment>
 </net>
 <net name="RXD" class="0">
@@
 <wire x1="198.12" y1="58.42" x2="193.04" y2="58.42" width="0.1524" layer="91"/>
 <label x="193.04" y="58.42" size="1.778" layer="91" rot="R180" xref="yes"/>
+</segment>
+<segment>
+<pinref part="U$1" gate="G$1" pin="DATA2-"/>
+<wire x1="218.44" y1="38.1" x2="228.6" y2="38.1" width="0.1524" layer="91"/>
+<label x="228.6" y="38.1" size="1.778" layer="91" xref="yes"/>
 </segment>
 </net>
@@
 <label x="193.04" y="66.04" size="1.778" layer="91" rot="R180" xref="yes"/>
 </segment>
+<segment>
+<pinref part="U$1" gate="G$1" pin="DATA1+"/>
+<wire x1="218.44" y1="35.56" x2="228.6" y2="35.56" width="0.1524" layer="91"/>
+<label x="228.6" y="35.56" size="1.778" layer="91" xref="yes"/>
+</segment>
 </net>
 <net name="TTL22" class="0">
@@
 <label x="193.04" y="63.5" size="1.778" layer="91" rot="R180" xref="yes"/>
 </segment>
-</net>
+<segment>
+<pinref part="U$1" gate="G$1" pin="DATA1-"/>
+<wire x1="218.44" y1="33.02" x2="231.14" y2="33.02" width="0.1524" layer="91"/>
+<label x="231.14" y="33.02" size="1.778" layer="91" xref="yes"/>
+</segment>
+</net>
