File: RPiOperant.brd (EAGLE design)
At the start: 136 x 100 mm, 62 parts, among them IC1 74LS14N, IC2 74LS14N, IC3 MCP3008, J1 USB_B_PTH, J2 POWER_JACK, J3 POWER_JACK, J4 USB_B_PTH, J5 1X2-3.5MM, J6 1X2-3.5MM, J7 1X2-3.5MM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

Commit message: new stuff!
Parts:
- removed J7, J8, J9: 1X2-3.5MM, adafruit:1X2-3.5MM
- added J10, J13, J14: (no value), SparkFun-Connectors:SCREWTERMINAL-3.5MM-3
- added J11, J12: (no value), SparkFun-Connectors:1X05
- added JP1: (no value), jumper:JP2
- added Q2, Q7: 60V/32A/35mΩ, SparkFun-DiscreteSemi:TO220V
- added R40, R41: 10K, resistor:0207/7
- moved R10 23.0 mm to (83.5, 62.9)
- moved R11 23.0 mm to (83.5, 72.9)
- moved R12 23.0 mm to (93.5, 67.9)
- moved R17 23.0 mm to (93.5, 72.9)
- moved R21 23.0 mm to (83.5, 67.9)
- moved R22 23.0 mm to (113.5, 72.9)
- moved R23 23.0 mm to (113.5, 67.9)
- moved R36 23.0 mm to (103.5, 72.9)
- moved R37 23.0 mm to (103.5, 67.9)
- moved R38 23.0 mm to (93.5, 62.9)
- moved R39 23.0 mm to (113.5, 62.9)
- moved R9 23.0 mm to (103.5, 62.9)
- moved U1 14.3 mm to (127.3, 77.1)
- moved J6 13.0 mm to (78.0, 4.00)
- moved J1 12.0 mm to (47.0, 10.0)
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Connections:
- removed net TEMP: X1.2
- new net DAT: J12.3
- new net LCCLK: J12.2
- new net TTL27: J10.1, Q2.2, R41.2
- new net YLW: J11.1
- net +3V3: now also J12.4
- net GND: now also J10.3, J12.1, J13.3, J14.3
- net GPIO17: now also J13.1; no longer J9.1
- net GPIO18: now also J13.2, X1.2; no longer J9.2
- net GPIO22: now also J10.2; no longer J8.2
- net GPIO27: now also Q2.3, R40.2; no longer J8.1
- net LOADCELLA+: now also J11.3
- net LOADCELLA-: now also J11.2
- net LOADCELLE+: now also J11.5
- net LOADCELLE-: now also J11.4
- net RPI_3.3V: now also JP1.1, Q2.1, R40.1
- net RPI_5V: now also JP1.2, JP1.3, R41.1
- net RXD: now also J14.2; no longer J7.2
- net TXD: now also J14.1; no longer J7.1
Other:
- board text added: "GENTNERLAB OPiRANT INTERFACE BRAD THEILMAN TIM SAINBURG"
- board text added: "GND"
- board text removed: "GENTNER LAB OPiRANT INTERFACE BRAD THEILMAN + TIM SAINBURG 2017"

Commit message: final draft
Parts:
- removed Q2, Q7: 60V/32A/35mΩ, SparkFun-DiscreteSemi:TO220V
- removed R40, R41: 10K, resistor:0207/7
- added B1: SPARKFUN_LOGIC_LEVEL_CONVERTER, SparkFun-Boards:SPARKFUN_LOGIC_LEVEL_CONVERTER
- added JP2, JP3, JP4: (no value), jumper:JP2
- moved JP1 24.0 mm to (122.0, 42.0)
- moved IC3 6.00 mm to (93.6, 54.1)
- moved Q5 4.12 mm to (71.0, 80.0)
- moved Q1 4.00 mm to (43.0, 80.0)
- moved Q3 4.00 mm to (29.0, 80.0)
- moved Q4 4.00 mm to (16.0, 80.0)
- moved Q6 4.00 mm to (57.0, 80.0)
- moved X1 4.00 mm to (41.0, 92.0)
- moved X2 4.00 mm to (97.0, 92.0)
- moved J4 1.41 mm to (64.0, 9.00)
- moved J1 1.00 mm to (47.0, 9.00)
Connections:
- new net N$22: B1.HV1, JP2.3
- new net N$23: B1.HV2, JP3.3
- new net N$32: J13.1, JP1.1
- new net N$33: J13.2, JP4.1
- new net TTL22: J10.2, JP3.2
- net +3V3: now also J12.5; no longer J12.4
- net +5V: now also J12.4
- net DAT: now also JP1.3
- net GND: now also B1.GND1, B1.GND2
- net GPIO17: now also JP1.2; no longer J13.1
- net GPIO18: now also JP4.2; no longer J13.2
- net GPIO22: now also B1.LV2, JP3.1; no longer J10.2
- net GPIO27: now also B1.LV1, JP2.1; no longer Q2.3, R40.2
- net LCCLK: now also JP4.3
- net RPI_3.3V: now also B1.LV; no longer JP1.1, Q2.1, R40.1
- net RPI_5V: now also B1.HV; no longer JP1.2, JP1.3, R41.1
- net TTL27: now also JP2.2; no longer Q2.2, R41.2
Routing:
- net +3V3: track 0.00 -> 341.3 mm, vias 0 -> 4
- net RPI_3.3V: track 0.00 -> 265.0 mm, vias 0 -> 6
- net CE1: track 0.00 -> 221.9 mm, vias 0 -> 5
- net GPIO27: track 0.00 -> 210.0 mm, vias 0 -> 3
- net RPI_5V: track 0.00 -> 208.9 mm, vias 0 -> 2
- net GPIO22: track 0.00 -> 201.8 mm, vias 0 -> 3
- net HOPPER_TRIG_GPIO: track 0.00 -> 197.0 mm, vias 0 -> 5
- net CENTER_PECK_GPIO: track 0.00 -> 196.5 mm, vias 0 -> 4
- net HOPPER_IR_GPIO: track 0.00 -> 196.1 mm, vias 0 -> 4
- net LEFT_PECK_GPIO: track 0.00 -> 194.3 mm, vias 0 -> 5
- net SCLK: track 0.00 -> 192.7 mm, vias 0 -> 4
- net AUX2: track 0.00 -> 190.2 mm, vias 0 -> 6
- net CE0: track 0.00 -> 188.1 mm, vias 0 -> 2
- net RIGHT_PECK_GPIO: track 0.00 -> 180.8 mm, vias 0 -> 2
- net IR_3: track 0.00 -> 176.7 mm, vias 0 -> 7
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Other:
- board text added: "/home/brad/Pictures/gentnerlab_logo_inverted.bmp"
- board text added: "3.3 5"
- board text added: "GPIO LC"

Commit message: alternate
Parts:
- removed IC3: MCP3008, adafruit:DIL16
- removed J1, J4: USB_B_PTH, SparkFun-Connectors:USB-B-PTH
- removed J5, J6: 1X2-3.5MM, adafruit:1X2-3.5MM
- added J15, J9: (no value), SparkFun-Connectors:SCREWTERMINAL-3.5MM-2
- added J7, J8: (no value), SparkFun-Connectors:1X04
- moved B1 57.2 mm to (63.0, 35.0)
- moved JP4 56.5 mm to (70.0, 14.0)
- moved JP1 56.1 mm to (70.0, 21.0)
- moved D1 49.7 mm to (46.0, 21.0)
- moved R2 34.9 mm to (21.0, 26.0)
- moved R26 31.6 mm to (21.0, 56.0)
- moved R24 29.2 mm to (45.0, 56.0)
- moved R16 26.3 mm to (9.00, 68.0)
- moved JP2 20.0 mm to (59.0, 21.0)
- moved JP3 19.4 mm to (59.0, 14.0)
- moved R14 19.0 mm to (21.0, 62.0)
- moved R5 18.6 mm to (45.0, 68.0)
- moved R25 18.0 mm to (33.0, 56.0)
- moved R7 17.8 mm to (33.0, 62.0)
- moved R3 17.2 mm to (33.0, 68.0)
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Connections:
- removed net ADC0: IC3.1, X1.1
- removed net ADC1: IC3.2, X2.14
- removed net ADC2: IC3.3, X2.7
- removed net ADC3: IC3.4, X2.6
- removed net ADC4: IC3.5, X2.5
- removed net ADC5: IC3.6
- removed net ADC6: IC3.7
- removed net ADC7: IC3.8
- removed net CE0: SV1.24, SV2.24
- removed net CE1: IC3.10, SV1.26, SV2.26
- removed net GPIO18: JP4.2, SV1.12, X1.2
- removed net MISO: IC3.12, SV1.21, SV2.21
- removed net MOSI: IC3.11, SV1.19, SV2.19
- removed net SCLK: IC3.13, SV1.23, SV2.23
- new net GPIO7: SV1.26, SV2.26
- new net GPIO8: JP4.2, SV1.24, SV2.24
- new net N$25: X2.7
- new net N$31: X2.6
- new net N$34: X2.5
- new net N$35: X2.14
- net +3V3: no longer IC3.15, IC3.16
- net AUX1: now also J9.1; no longer J5.1, SV1.7
- net AUX2: now also J9.2; no longer J5.2
- net AUX3: now also J15.1; no longer J6.1
- net AUX4: now also J15.2; no longer J6.2
- net GND: now also J7.4, J8.4; no longer IC3.14, IC3.9, J1.GND, J1.SHLD1, J1.SHLD2, J4.GND, J4.SHLD1, J4.SHLD2
- net IR_4_GPIO: now also SV1.21, SV2.21; no longer SV1.38
- net IR_5_GPIO: now also SV1.23, SV2.23; no longer SV1.40
- net IR_6_GPIO: now also SV1.19, SV2.19; no longer SV1.35, SV2.35
- net TTL22: now also X1.2
- net TTL27: now also X1.1
- net USB1_D+: now also J7.3; no longer J1.D+
- net USB1_D-: now also J7.2; no longer J1.D-
- net USB1_VBUS: now also J7.1; no longer J1.VBUS
- net USB2_D+: now also J8.3; no longer J4.D+
- net USB2_D-: now also J8.2; no longer J4.D-
- net USB2_VBUS: now also J8.1; no longer J4.VBUS
Routing:
- net CE1: track 221.9 -> 0.00 mm, vias 5 -> 0
- net SCLK: track 192.7 -> 0.00 mm, vias 4 -> 0
- net CE0: track 188.1 -> 0.00 mm, vias 2 -> 0
- net MISO: track 176.3 -> 0.00 mm, vias 6 -> 0
- net GPIO7: track 0.00 -> 162.8 mm, vias 0 -> 1
- net MOSI: track 152.9 -> 0.00 mm, vias 5 -> 0
- net GPIO8: track 0.00 -> 145.0 mm, vias 0 -> 3
- net GPIO18: track 137.5 -> 0.00 mm, vias 2 -> 0
- net TTL22: track 44.6 -> 170.9 mm, vias 1 -> 4
- net IR_4_GPIO: track 79.1 -> 169.3 mm, vias 3 -> 6
- net TTL27: track 53.1 -> 140.7 mm, vias 0 -> 2
- net ADC0: track 78.4 -> 0.00 mm, vias 1 -> 0
- net IR_3: track 176.7 -> 102.3 mm, vias 7 -> 3
- net AUX1: track 169.4 -> 98.7 mm, vias 6 -> 3
- net RPI_3.3V: track 265.0 -> 197.8 mm, vias 6 -> 4
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Other:
- board text added: "3.3V 5V"
- board text added: "GPIO8"
- board text added: "RASPBERRY PI"
- board text added: "Rev. A 2017"
- board text removed: "3.3 5"
- board text removed: "GPIO18"

Commit message: final draft
Parts:
- added J1: (no value), SparkFun-Connectors:SCREWTERMINAL-3.5MM-4
- moved JP4 17.0 mm to (78.0, 29.0)
- moved J15 15.0 mm to (72.0, 4.00)
- moved J9 15.0 mm to (64.0, 4.00)
- moved JP3 12.0 mm to (67.0, 23.0)
- moved JP1 8.25 mm to (78.0, 23.0)
- moved J8 8.00 mm to (50.0, 3.00)
- moved J7 7.00 mm to (37.0, 3.00)
- moved J2 4.47 mm to (27.0, -2.00)
- moved J3 3.61 mm to (15.0, -2.00)
- moved J11 3.16 mm to (89.4, 30.2)
- moved J12 3.16 mm to (117.3, 30.2)
- moved JP2 2.24 mm to (58.0, 23.0)
- moved B1 1.00 mm to (63.0, 36.0)
Connections:
- removed net N$25: X2.7
- removed net N$31: X2.6
- removed net N$34: X2.5
- removed net N$35: X2.14
- new net AUX5: J1.1, X2.5
- new net AUX6: J1.2, X2.6
- new net AUX7: J1.3, X2.7
- new net AUX8: J1.4, X2.14
Routing:
- net AUX5: track 0.00 -> 111.4 mm, vias 0 -> 5
- net AUX8: track 0.00 -> 110.5 mm, vias 0 -> 2
- net AUX7: track 0.00 -> 104.0 mm, vias 0 -> 2
- net AUX6: track 0.00 -> 95.9 mm, vias 0 -> 4
- net N$2: track 45.5 -> 122.1 mm, vias 4 -> 0
- net IR_1: track 193.6 -> 130.3 mm, vias 3 -> 2
- net USB2_D-: track 108.0 -> 170.2 mm, vias 4 -> 3
- net RGB_CUE_B: track 98.5 -> 154.0 mm, vias 1 -> 3
- net RIGHT_PECK_GPIO: track 182.0 -> 229.4 mm, vias 2 -> 4
- net HOPPER_IR_GPIO: track 173.1 -> 220.1 mm, vias 4 -> 6
- net N$5: track 84.3 -> 129.6 mm, vias 4 -> 0
- net AUX2: track 152.7 -> 188.7 mm, vias 3 -> 4
- net LCCLK: track 70.2 -> 38.4 mm, vias 1 -> 0
- net USB1_D+: track 117.5 -> 148.5 mm, vias 3 -> 1
- net +3V3: track 328.9 -> 299.4 mm
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Other:
- board text added: "AUX5"
- board text added: "AUX6"
- board text added: "AUX7"
- board text added: "AUX8"
- board text added: "HX711 LOAD CELL AMPLIFIER"
- board text added: "LOAD CELL SELECT"
- board text added: "TTL SELECT"
- board text added: "TTL22"
- board text added: "TTL27"
- board text removed: "GPIO22"
- board text removed: "GPIO27"

Commit message: Revision A
Routing:
- net GND: track 30.8 -> 583.7 mm, vias 0 -> 3
- net IR_3_GPIO: track 161.1 -> 262.9 mm, vias 4 -> 3
- net LOADCELLA-: track 105.3 -> 198.4 mm, vias 1 -> 3
- net LOADCELLA+: track 95.5 -> 186.8 mm, vias 6 -> 0
- net N$5: track 129.6 -> 47.7 mm
- net N$2: track 122.1 -> 44.2 mm
- net RIGHT_LED: track 74.7 -> 150.7 mm, vias 3 -> 0
- net TTL27: track 150.0 -> 223.9 mm, vias 2 -> 4
- net GPIO8: track 141.6 -> 197.8 mm
- net IR_3: track 106.9 -> 155.1 mm, vias 3 -> 5
- net AUX8: track 110.5 -> 157.4 mm
- net GPIO22: track 157.7 -> 201.1 mm
- net HOPPER: track 77.5 -> 119.4 mm, vias 2 -> 0
- net GPIO17: track 161.4 -> 199.2 mm, vias 4 -> 7
- net N$30: track 53.2 -> 90.9 mm, vias 2 -> 3
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- removed copper zone on layer 16, net GND

Commit message: revision b
Parts:
- removed SV2: (no value), con-lstb:MA20-2
- added SV3: (no value), con-lstb:MA20-2
- moved SV1 4.00 mm to (131.0, 38.0)
Connections:
- removed net CENTNER_IR: R5.1, R6.1
- new net GPIO4: SV1.7, SV3.7
- new net ID_SC: SV1.28, SV3.28
- new net ID_SD: SV1.27, SV3.27
- new net PCM_CLK: SV1.12, SV3.12
- new net PCM_DIN: SV1.38, SV3.38
- new net PCM_DOUT: SV1.40, SV3.40
- new net PCM_FS: SV1.35, SV3.35
- net AUX2: now also SV3.32
- net CENTER_IR: now also R5.1, R6.1
- net CENTER_PECK_GPIO: now also SV3.33; no longer SV2.33
- net GND: now also SV3.14, SV3.20, SV3.25, SV3.30, SV3.34, SV3.39, SV3.6, SV3.9; no longer SV2.14, SV2.20, SV2.25, SV2.30, SV2.34, SV2.39, SV2.6, SV2.9
- net GPIO17: now also SV3.11; no longer SV2.11
- net GPIO22: now also SV3.15; no longer SV2.15
- net GPIO27: now also SV3.13; no longer SV2.13
- net GPIO7: now also SV3.26; no longer SV2.26
- net GPIO8: now also SV3.24; no longer SV2.24
- net HOPPER_IR_GPIO: now also SV3.29; no longer SV2.29
- net HOPPER_TRIG_GPIO: now also SV3.36; no longer SV2.36
- net IR_1_GPIO: now also SV3.16
- net IR_2_GPIO: now also SV3.18; no longer SV2.18
- net IR_3_GPIO: now also SV3.22; no longer SV2.22
- net IR_4_GPIO: now also SV3.21; no longer SV2.21
- net IR_5_GPIO: now also SV3.23; no longer SV2.23
- net IR_6_GPIO: now also SV3.19; no longer SV2.19
- net LEFT_PECK_GPIO: now also SV3.31; no longer SV2.31
- net RIGHT_PECK_GPIO: now also SV3.37; no longer SV2.37
- net RPI_3.3V: now also SV3.1, SV3.17; no longer SV2.1, SV2.17
- net RPI_5V: now also SV3.2, SV3.4; no longer SV2.2, SV2.4
- net RXD: now also SV3.10
- net SCL: now also SV3.5
- net SDA: now also SV3.3
- net TXD: now also SV3.8
Routing:
- net GND: track 583.7 -> 0.00 mm, vias 3 -> 0
- net +3V3: track 291.8 -> 0.00 mm, vias 6 -> 0
- net IR_3_GPIO: track 262.9 -> 0.00 mm, vias 3 -> 0
- net RIGHT_PECK_GPIO: track 252.8 -> 0.00 mm, vias 5 -> 0
- net HOPPER_IR_GPIO: track 230.6 -> 0.00 mm, vias 10 -> 0
- net CENTER_PECK_GPIO: track 229.9 -> 0.00 mm, vias 6 -> 0
- net TTL27: track 223.9 -> 0.00 mm, vias 4 -> 0
- net RPI_3.3V: track 214.6 -> 0.00 mm, vias 6 -> 0
- net HOPPER_TRIG_GPIO: track 209.6 -> 0.00 mm, vias 7 -> 0
- net GPIO22: track 201.1 -> 0.00 mm, vias 3 -> 0
- net GPIO17: track 199.2 -> 0.00 mm, vias 7 -> 0
- net LOADCELLA-: track 198.4 -> 0.00 mm, vias 3 -> 0
- net GPIO8: track 197.8 -> 0.00 mm, vias 4 -> 0
- net LEFT_PECK_GPIO: track 196.4 -> 0.00 mm, vias 7 -> 0
- net IR_2: track 194.4 -> 0.00 mm, vias 2 -> 0
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
Commit message: updates
Parts:
- removed J3: POWER_JACK, SparkFun-Connectors:POWER_JACK_PTH
- removed R18: 10k, resistor:0207/7
- removed R19: 20k, resistor:0207/7
- added C1: 100nF, adafruit:C050-025X075
- added C2, C3, C4: 10uF, adafruit:C050-025X075
- added U$1: V_REG_LD1117VXX, SparkFun-IC-Power:78XXL
- added U2: (no value), SparkFun-IC-Power:TO-220-ALT
- moved J2 139.0 mm to (166.0, -4.00)
- moved R16 121.0 mm to (97.0, -15.0)
- moved D1 107.3 mm to (151.0, 43.0), turned to 90 degrees
- moved B1 63.9 mm to (14.0, 77.0)
- moved Q4 53.6 mm to (62.0, 92.0)
- moved Q1 52.6 mm to (89.0, 92.0)
- moved Q3 52.6 mm to (75.0, 92.0)
- moved Q5 51.7 mm to (116.0, 92.0)
- moved Q6 51.7 mm to (102.0, 92.0)
- moved IC1 36.9 mm to (36.0, 88.0)
- moved J7 35.0 mm to (65.0, -18.0)
- moved J8 35.0 mm to (78.0, -18.0)
- moved IC2 33.1 mm to (61.0, 83.0)
- moved R1 14.6 mm to (17.0, 54.0)
- moved R13 14.6 mm to (41.0, 48.0)
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Connections:
- new net 5V: C4.1, U2.OUT
- net +3V3: now also C2.1, U$1.GND; no longer R18.1, R19.2
- net +5V: no longer J3.PWR, R18.2
- net 12V: now also C1.1, C3.1, U$1.OUT, U2.IN
- net GND: now also C1.2, C2.2, C3.2, C4.2, U$1.IN, U2.GND; no longer J3.GND, J3.GNDBREAK, R19.1
Other:
- board size 136 x 100 mm -> 136 x 112 mm

Commit message: version 2
Parts:
- removed C3, C4: 10uF, adafruit:C050-025X075
- removed U2: (no value), SparkFun-IC-Power:TO-220-ALT
- moved J2 151.0 mm to (15.0, -3.00)
- moved R22 97.9 mm to (16.0, 53.0)
- moved R23 97.8 mm to (16.0, 49.0)
- moved U$1 96.5 mm to (55.0, 41.0)
- moved R9 87.9 mm to (16.0, 61.0)
- moved R39 85.9 mm to (28.0, 61.0)
- moved B1 85.1 mm to (95.0, 51.0)
- moved D1 84.2 mm to (72.0, 72.0), turned to 270 degrees
- moved R37 75.9 mm to (28.0, 49.0)
- moved R16 73.2 mm to (115.0, 56.0)
- moved R11 67.6 mm to (16.0, 57.0)
- moved R17 65.6 mm to (28.0, 57.0)
- moved R36 63.6 mm to (40.0, 57.0)
- moved IC1 61.2 mm to (74.0, 40.0)
- moved Q5 58.5 mm to (61.0, 72.0)
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Connections:
- removed net 5V: C4.1, U2.OUT
- net 12V: now also X1.23; no longer C3.1, U2.IN
- net GND: no longer C3.2, C4.2, U2.GND, X1.23
Other:
- board size 136 x 112 mm -> 136 x 94 mm
